File: CustomBoot32/CustomBoot32.kicad_sch (KiCad schematic)
At the start: 43 parts, among them J1 USB_B_Micro, J2 Conn_01x27_Pin, Q1 SS8050, Q2 SS8050, SW1 SW_Push, SW2 SW_Push, U1 ESP32-WROOM-32D, U2 STM32F103C8Tx, U3 AMS1117-3.3, U4 CP2102N-Axx-xQFN28, Y1 GND24

Commit message: Updated
Parts:
- removed R9: 4k7, symbol Device:R
- added R10: 10k, Resistor_SMD:R_0402_1005Metric, symbol Device:R
- added SW3: SW_SPDT, Button_Switch_SMD:SW_SPDT_PCM12, symbol Switch:SW_SPDT
- J2: footprint (none) -> Connector:FanPinHeader_1x04_P2.54mm_Vertical
- renumbered C11 to C17
Connections:
- net 3.3(AMS): now also SW3.3 (C)
- net BOOT0: now reaches U2.44 (BOOT0)
- net BOOT0: now also R10.1
- new net: R10.2, SW3.2 (B)
